File: hw/kicad/MotCtrl.sch (KiCad schematic (older format))
At the start: 3 parts

Commit message: Annotation
Parts:
- gave numbers to parts that had none: 3
Changed lines of the file:
@@
 	6050 5050 6950 5050
 $Comp
-L TESTPAD TP?
+L TESTPAD TP1
 U 1 1 581F3C20
 P 9250 3250
-F 0 "TP?" V 9200 3200 40  0000 C CNN
+F 0 "TP1" V 9200 3200 40  0000 C CNN
 F 1 "Phase A" V 9250 3500 40  0000 C CNN
 F 2 "Wire_Pads:SolderWirePad_single_SMD_5x10mm" V 9250 3400 60  0001 C CNN
@@
 	9200 3350 8450 3350
 $Comp
-L TESTPAD TP?
+L TESTPAD TP2
 U 1 1 581F8700
 P 9250 3350
-F 0 "TP?" V 9200 3300 40  0000 C CNN
+F 0 "TP2" V 9200 3300 40  0000 C CNN
 F 1 "Phase B" V 9250 3600 40  0000 C CNN
 F 2 "Wire_Pads:SolderWirePad_single_SMD_5x10mm" V 9250 3500 60  0001 C CNN
@@
 $EndComp
 $Comp
-L TESTPAD TP?
+L TESTPAD TP3
 U 1 1 581F8822
 P 9250 3450
-F 0 "TP?" V 9200 3400 40  0000 C CNN
+F 0 "TP3" V 9200 3400 40  0000 C CNN
 F 1 "Phase C" V 9250 3700 40  0000 C CNN
 F 2 "Wire_Pads:SolderWirePad_single_SMD_5x10mm" V 9250 3600 60  0001 C CNN

Commit message: Aligned, started rework current shunt layout and copper pour
Parts:
- TP1, TP2, TP3: footprint Wire_Pads:SolderWirePad_single_SMD_5x10mm -> pads:SolderWirePad_single_SMD_5x5mm
Changed lines of the file:
@@
 F 0 "TP1" V 9200 3200 40  0000 C CNN
 F 1 "Phase A" V 9250 3500 40  0000 C CNN
-F 2 "Wire_Pads:SolderWirePad_single_SMD_5x10mm" V 9250 3400 60  0001 C CNN
+F 2 "pads:SolderWirePad_single_SMD_5x5mm" V 9250 3400 60  0001 C CNN
 F 3 "" V 9250 3400 60  0000 C CNN
 	1    9250 3250
@@
 F 0 "TP2" V 9200 3300 40  0000 C CNN
 F 1 "Phase B" V 9250 3600 40  0000 C CNN
-F 2 "Wire_Pads:SolderWirePad_single_SMD_5x10mm" V 9250 3500 60  0001 C CNN
+F 2 "pads:SolderWirePad_single_SMD_5x5mm" V 9250 3500 60  0001 C CNN
 F 3 "" V 9250 3500 60  0000 C CNN
 	1    9250 3350
@@
 F 0 "TP3" V 9200 3400 40  0000 C CNN
 F 1 "Phase C" V 9250 3700 40  0000 C CNN
-F 2 "Wire_Pads:SolderWirePad_single_SMD_5x10mm" V 9250 3600 60  0001 C CNN
+F 2 "pads:SolderWirePad_single_SMD_5x5mm" V 9250 3600 60  0001 C CNN
 F 3 "" V 9250 3600 60  0000 C CNN
 	1    9250 3450
